File: tests/repros/smt-pill-pad-roundrect.kicad_pcb (KiCad board)
At the start: 2 copper layers, 5 parts

Commit message: up
Other:
- board outline added: 8 x 8 mm
Changed lines of the file:
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@@
     (net 0)
   )
+  (gr_line
+    (start 96 96)
+    (end 104 96)
+    (stroke
+      (width 0.1)
+      (type default)
+    )
+    (layer Edge.Cuts)
+  )
+  (gr_line
+    (start 104 96)
+    (end 104 104)
+    (stroke
+      (width 0.1)
+      (type default)
+    )
+    (layer Edge.Cuts)
+  )
+  (gr_line
+    (start 104 104)
+    (end 96 104)
+    (stroke
+      (width 0.1)
+      (type default)
+    )
+    (layer Edge.Cuts)
+  )
+  (gr_line
+    (start 96 104)
+    (end 96 96)
+    (stroke
+      (width 0.1)
+      (type default)
+    )
+    (layer Edge.Cuts)
+  )
 )
